File: panel_light_control.kicad_pcb (KiCad board)
At the start: 4 copper layers, 109 parts, among them J1 Conn_01x02, J10 Conn_01x09, J11 RJ45_Shielded, J12 RJ45_Shielded, J13 HR911105A, J2 Conn_01x02, J3 Conn_01x02, J4 Conn_01x04, J5 Conn_01x06, J6 Conn_01x04, J7 Conn_01x04, J8 Conn_01x07, J9 Conn_01x06, Q1 IRF540N, Q2 IRF540N, Q3 IRF540N, U1 L7805, U2 LM324, U3 STM32F207VGTx, U4 MCP2562-E-P, U5 LAN8720A, Y1 Crystal_GND24

Commit message: Finished initial PHY-magjack routing.
Parts:
- J6: footprint Connector_JST:JST_PH_S4B-PH-K_1x04_P2.00mm_Horizontal -> TerminalBlock_Phoenix:TerminalBlock_Phoenix_MKDS-1,5-4_1x04_P5.00mm_Horizontal
- moved C34 44.2 mm to (87.2, 95.5)
- moved U4 44.2 mm to (84.8, 101.3)
- moved J11 43.2 mm to (62.4, 111.6)
- moved J12 43.2 mm to (62.4, 92.2)
- moved R30 43.2 mm to (73.3, 98.3)
- moved C30 43.2 mm to (73.4, 93.9)
- moved U1 42.6 mm to (95.9, 80.1), turned to 270 degrees
- moved C20 36.9 mm to (126.2, 123.0), turned to 0 degrees
- moved C38 33.0 mm to (77.2, 135.4)
- moved C22 32.6 mm to (123.6, 117.4), turned to 90 degrees
- moved C17 32.2 mm to (123.5, 140.8), turned to 270 degrees
- moved R21 31.4 mm to (127.3, 126.0)
- moved C12 31.3 mm to (102.7, 84.3), turned to 90 degrees
- moved Y1 30.4 mm to (121.0, 116.8), turned to 270 degrees
- moved C19 30.1 mm to (121.9, 140.8), turned to 270 degrees
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Connections:
- net Net-(J13-Pad1) renamed /MCU/TX_P
- net Net-(J13-Pad2) renamed /MCU/TX_N
- net Net-(J13-Pad3) renamed /MCU/RX_P
- net Net-(J13-Pad6) renamed /MCU/RX_N
Routing:
- net VDDA: track 0.00 -> 45.3 mm, vias 0 -> 1
- net /MCU/RX_N: track 0.00 -> 37.6 mm
- net /MCU/RX_P: track 0.00 -> 33.5 mm
- net Net-(R31-Pad1): track 0.00 -> 30.4 mm, vias 0 -> 2
- net Net-(R35-Pad2): track 0.00 -> 29.9 mm, vias 0 -> 2
- net /MCU/TX_P: track 0.00 -> 18.5 mm
- net +3.3V: track 0.00 -> 18.2 mm
- net GND: track 0.00 -> 16.4 mm, vias 0 -> 14
- net /MCU/TX_N: track 0.00 -> 15.5 mm
- net Net-(R27-Pad1): track 0.00 -> 13.4 mm
- net Net-(R26-Pad1): track 0.00 -> 11.4 mm
- net Net-(R25-Pad1): track 0.00 -> 7.13 mm
- net Net-(R24-Pad1): track 0.00 -> 6.71 mm
- net Net-(R23-Pad1): track 0.00 -> 6.40 mm
- net Net-(R22-Pad1): track 0.00 -> 5.95 mm
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
Commit message: schematic clean-up, BOM info partially added
Parts:
- removed J4: Conn_01x04, Connector_JST:JST_PH_S4B-PH-K_1x04_P2.00mm_Horizontal
- removed J9: Conn_01x06, Connector_JST:JST_PH_S6B-PH-K_1x06_P2.00mm_Horizontal
- added I2C1: Conn_01x04, Connector_JST:JST_PH_S4B-PH-K_1x04_P2.00mm_Horizontal, F.Cu at (122.8, 157.0)
- added JTAG1: Conn_01x06, Connector_JST:JST_PH_S6B-PH-K_1x06_P2.00mm_Horizontal, F.Cu at (134.4, 157.0)
- moved C13 105.0 mm to (35.1, 120.7), turned to 0 degrees
- moved R34 9.36 mm to (79.0, 116.2), turned to 270 degrees
- moved R32 7.59 mm to (77.3, 116.2), turned to 270 degrees
- moved R38 6.17 mm to (75.7, 116.2), turned to 270 degrees
- moved R37 5.39 mm to (74.1, 116.2), turned to 270 degrees
- renumbered J5 to DBG1, J2 to PANEL1, J3 to PANEL2, J10 to SPI0, J8 to SPI1, J7 to UART1
Connections:
- J13 pad 12: LED_GRN- -> LED_YLW-
- J13 pad 9: LED_YLW- -> LED_GRN-
Routing:
- net VDDA: track 45.3 -> 0.00 mm, vias 1 -> 0
- net /MCU/RX_N: track 37.6 -> 0.00 mm
- net /MCU/RX_P: track 33.5 -> 0.00 mm
- net Net-(R31-Pad1): track 30.4 -> 0.00 mm, vias 2 -> 0
- net Net-(R35-Pad2): track 29.9 -> 0.00 mm, vias 2 -> 0
- net /MCU/TX_P: track 18.5 -> 0.00 mm
- net +3.3V: track 18.2 -> 0.00 mm
- net GND: track 16.4 -> 0.00 mm, vias 14 -> 0
- net /MCU/TX_N: track 15.5 -> 0.00 mm
- net Net-(R27-Pad1): track 13.4 -> 0.00 mm
- net Net-(R26-Pad1): track 11.4 -> 0.00 mm
- net Net-(R25-Pad1): track 7.13 -> 0.00 mm
- net Net-(R24-Pad1): track 6.71 -> 0.00 mm
- net Net-(R23-Pad1): track 6.40 -> 0.00 mm
- net Net-(R22-Pad1): track 5.95 -> 0.00 mm
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