File: panel_light_control.kicad_pcb (KiCad board)
At the start: 4 copper layers, 90 x 100 mm, 161 parts, among them J1 Conn_01x02, J11 RJ45_Shielded, J13 HR911105A, J2 RJ45_Shielded, J6 Conn_01x04, Q1 IRF540N, Q2 IRF540N, Q3 IRF540N, U1 L7805, U2 LM324, U3 STM32F207VGT6, U4 MCP2562-E-P, U5 LAN8742A, Y1 Crystal_GND24

Commit message: BOM DONE
Parts:
- C1, C32, C35, C8, C9: value 1uF -> 2.2uF
- C33: value 470pF -> 10nF
- R1, R7, R9: value 30k -> 33k
- R13, R15, R4: value 100 -> 120R
- R14, R16, R5: value 2k -> 2.2k
- R19, R20, R22, R23, R24, R25, R26: value 10R -> 22R
- R28, R29: value 10k -> 12k
- R35, R36: value 330R -> 1k
- R39, R48: value 220R -> 120R
- R54: value 100R -> 120R
Changed lines of the file:
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@@
       (effects (font (size 1 1) (thickness 0.15)))
     )
-    (fp_text value 100R (at 0 1.43 90) (layer F.Fab)
+    (fp_text value 120R (at 0 1.43 90) (layer F.Fab)
       (effects (font (size 1 1) (thickness 0.15)))
     )
@@
       (effects (font (size 1 1) (thickness 0.15)))
     )
-    (fp_text value 220R (at 0 1.43) (layer F.Fab)
+    (fp_text value 120R (at 0 1.43) (layer F.Fab)
       (effects (font (size 1 1) (thickness 0.15)))
     )
@@
       (effects (font (size 1 1) (thickness 0.15)))
     )
-    (fp_text value 220R (at 0 1.43 270) (layer F.Fab)
+    (fp_text value 120R (at 0 1.43 270) (layer F.Fab)
       (effects (font (size 1 1) (thickness 0.15)))
     )
@@
       (effects (font (size 1 1) (thickness 0.15)))
     )
-    (fp_text value 2k (at 0 1.43 90) (layer F.Fab)
+    (fp_text value 2.2k (at 0 1.43 90) (layer F.Fab)
       (effects (font (size 1 1) (thickness 0.15)))
     )
@@
       (effects (font (size 1 1) (thickness 0.15)))
     )
-    (fp_text value 2k (at 0 1.43 90) (layer F.Fab)
+    (fp_text value 2.2k (at 0 1.43 90) (layer F.Fab)
       (effects (font (size 1 1) (thickness 0.15)))
     )
@@
       (effects (font (size 1 1) (thickness 0.15)))
     )
-    (fp_text value 2k (at 0 1.43) (layer F.Fab)
+    (fp_text value 2.2k (at 0 1.43) (layer F.Fab)
       (effects (font (size 1 1) (thickness 0.15)))
     )
@@
       (effects (font (size 1 1) (thickness 0.15)))
     )
-    (fp_text value 100 (at 0 1.43 270) (layer F.Fab)
+    (fp_text value 120R (at 0 1.43 270) (layer F.Fab)
       (effects (font (size 1 1) (thickness 0.15)))
     )
@@
       (effects (font (size 1 1) (thickness 0.15)))
     )
-    (fp_text value 30k (at 0 1.43 90) (layer F.Fab)
+    (fp_text value 33k (at 0 1.43 90) (layer F.Fab)
       (effects (font (size 1 1) (thickness 0.15)))
     )
@@
       (effects (font (size 1 1) (thickness 0.15)))
     )
-    (fp_text value 100 (at 0 1.43 270) (layer F.Fab)
+    (fp_text value 120R (at 0 1.43 270) (layer F.Fab)
       (effects (font (size 1 1) (thickness 0.15)))
     )
@@
       (effects (font (size 1 1) (thickness 0.15)))
     )
-    (fp_text value 30k (at 0 1.43 90) (layer F.Fab)
+    (fp_text value 33k (at 0 1.43 90) (layer F.Fab)
       (effects (font (size 1 1) (thickness 0.15)))
     )
@@
       (effects (font (size 1 1) (thickness 0.15)))
     )
-    (fp_text value 1uF (at 0 1.43 90) (layer F.Fab)
+    (fp_text value 2.2uF (at 0 1.43 90) (layer F.Fab)
       (effects (font (size 1 1) (thickness 0.15)))
     )
@@
       (effects (font (size 1 1) (thickness 0.15)))
     )
-    (fp_text value 1uF (at 0 1.43 90) (layer F.Fab)
+    (fp_text value 2.2uF (at 0 1.43 90) (layer F.Fab)
       (effects (font (size 1 1) (thickness 0.15)))
     )
@@
       (effects (font (size 1 1) (thickness 0.15)))
     )
-    (fp_text value 1uF (at 0 1.43 270) (layer F.Fab)
+    (fp_text value 2.2uF (at 0 1.43 270) (layer F.Fab)
       (effects (font (size 1 1) (thickness 0.15)))
     )
@@
       (effects (font (size 1 1) (thickness 0.15)))
     )
-    (fp_text value 10R (at 0 1.43) (layer F.Fab)
+    (fp_text value 22R (at 0 1.43) (layer F.Fab)
       (effects (font (size 1 1) (thickness 0.15)))
     )
@@
       (effects (font (size 1 1) (thickness 0.15)))
     )
-    (fp_text value 10R (at 0 1.43) (layer F.Fab)
+    (fp_text value 22R (at 0 1.43) (layer F.Fab)
       (effects (font (size 1 1) (thickness 0.15)))
     )
@@
       (effects (font (size 1 1) (thickness 0.15)))
     )
-    (fp_text value 1uF (at 0 1.43 270) (layer F.Fab)
+    (fp_text value 2.2uF (at 0 1.43 270) (layer F.Fab)
       (effects (font (size 1 1) (thickness 0.15)))
     )
@@
       (effects (font (size 1 1) (thickness 0.15)))
     )
-    (fp_text value 470pF (at 0 1.43 180) (layer F.Fab)
+    (fp_text value 10nF (at 0 1.43 180) (layer F.Fab)
       (effects (font (size 1 1) (thickness 0.15)))
     )
@@
       (effects (font (size 1 1) (thickness 0.15)))
     )
-    (fp_text value 1uF (at 0 1.43 180) (layer F.Fab)
+    (fp_text value 2.2uF (at 0 1.43 180) (layer F.Fab)
       (effects (font (size 1 1) (thickness 0.15)))
     )
@@
       (effects (font (size 1 1) (thickness 0.15)))
     )
-    (fp_text value 30k (at 0 1.43 90) (layer F.Fab)
+    (fp_text value 33k (at 0 1.43 90) (layer F.Fab)
       (effects (font (size 1 1) (thickness 0.15)))
     )
@@
       (effects (font (size 1 1) (thickness 0.15)))
     )
-    (fp_text value 100 (at 0 1.43 270) (layer F.Fab)
+    (fp_text value 120R (at 0 1.43 270) (layer F.Fab)
       (effects (font (size 1 1) (thickness 0.15)))
     )
@@
       (effects (font (size 1 1) (thickness 0.15)))
     )
-    (fp_text value 10R (at 0 1.43 225) (layer F.Fab)
+    (fp_text value 22R (at 0 1.43 225) (layer F.Fab)
       (effects (font (size 1 1) (thickness 0.15)))
     )
@@
       (effects (font (size 1 1) (thickness 0.15)))
     )
-    (fp_text value 10R (at 0 1.43 225) (layer F.Fab)
+    (fp_text value 22R (at 0 1.43 225) (layer F.Fab)
       (effects (font (size 1 1) (thickness 0.15)))
     )
@@
       (effects (font (size 1 1) (thickness 0.15)))
     )
-    (fp_text value 10R (at 0 1.43) (layer F.Fab)
+    (fp_text value 22R (at 0 1.43) (layer F.Fab)
       (effects (font (size 1 1) (thickness 0.15)))
     )
@@
       (effects (font (size 1 1) (thickness 0.15)))
     )
-    (fp_text value 10R (at 0 1.43) (layer F.Fab)
+    (fp_text value 22R (at 0 1.43) (layer F.Fab)
       (effects (font (size 1 1) (thickness 0.15)))
     )
@@
       (effects (font (size 1 1) (thickness 0.15)))
     )
-    (fp_text value 10R (at 0 1.43) (layer F.Fab)
+    (fp_text value 22R (at 0 1.43) (layer F.Fab)
       (effects (font (size 1 1) (thickness 0.15)))
     )
@@
       (effects (font (size 1 1) (thickness 0.15)))
     )
-    (fp_text value 10k (at 0 1.43) (layer F.Fab)
+    (fp_text value 12k (at 0 1.43) (layer F.Fab)
       (effects (font (size 1 1) (thickness 0.15)))
     )
@@
       (effects (font (size 1 1) (thickness 0.15)))
     )
-    (fp_text value 10k (at 0 1.43) (layer F.Fab)
+    (fp_text value 12k (at 0 1.43) (layer F.Fab)
       (effects (font (size 1 1) (thickness 0.15)))
     )
@@
       (effects (font (size 1 1) (thickness 0.15)))
     )
-    (fp_text value 330R (at 0 1.43 90) (layer F.Fab)
+    (fp_text value 1k (at 0 1.43 90) (layer F.Fab)
       (effects (font (size 1 1) (thickness 0.15)))
     )
@@
       (effects (font (size 1 1) (thickness 0.15)))
     )
-    (fp_text value 330R (at 0 1.43 90) (layer F.Fab)
+    (fp_text value 1k (at 0 1.43 90) (layer F.Fab)
       (effects (font (size 1 1) (thickness 0.15)))
     )
@@
   (segment (start 137.338 99.949) (end 137.338 109.6135) (width 0.2) (layer F.Cu) (net 72))
   (segment (start 137.338 109.6135) (end 136.876388 110.075112) (width 0.2) (layer F.Cu) (net 72))
-  (segment (start 140.62646 115.97398) (end 141.57646 115.97398) (width 0.2) (layer F.Cu) (net 170))
-  (segment (start 139.90498 115.2525) (end 140.62646 115.97398) (width 0.2) (layer F.Cu) (net 170))
-  (segment (start 139.065 94.89948) (end 139.065 110.109) (width 0.2) (layer F.Cu) (net 170))
-  (segment (start 137.37844 93.21292) (end 139.065 94.89948) (width 0.2) (layer F.Cu) (net 170))
-  (segment (start 139.065 110.109) (end 138.2395 110.9345) (width 0.2) (layer F.Cu) (net 170))
-  (segment (start 138.2395 110.9345) (end 138.2395 114.808) (width 0.2) (layer F.Cu) (net 170))
-  (segment (start 138.2395 114.808) (end 138.684 115.2525) (width 0.2) (layer F.Cu) (net 170))
-  (segment (start 138.684 115.2525) (end 139.90498 115.2525) (width 0.2) (layer F.Cu) (net 170))
   (segment (start 132.6055 96.0264) (end 133.118 96.0264) (width 0.25) (layer F.Cu) (net 73))
   (segment (start 133.92079 95.22361) (end 133.92079 94.42521) (width 0.25) (layer F.Cu) (net 73))
@@
   (segment (start 132.618989 92.740989) (end 131.666489 92.740989) (width 0.2) (layer B.Cu) (net 169))
   (segment (start 135.89 101.7905) (end 135.89 96.012) (width 0.2) (layer B.Cu) (net 169))
+  (segment (start 140.62646 115.97398) (end 141.57646 115.97398) (width 0.2) (layer F.Cu) (net 170))
+  (segment (start 139.90498 115.2525) (end 140.62646 115.97398) (width 0.2) (layer F.Cu) (net 170))
+  (segment (start 139.065 94.89948) (end 139.065 110.109) (width 0.2) (layer F.Cu) (net 170))
+  (segment (start 137.37844 93.21292) (end 139.065 94.89948) (width 0.2) (layer F.Cu) (net 170))
+  (segment (start 139.065 110.109) (end 138.2395 110.9345) (width 0.2) (layer F.Cu) (net 170))
+  (segment (start 138.2395 110.9345) (end 138.2395 114.808) (width 0.2) (layer F.Cu) (net 170))
+  (segment (start 138.2395 114.808) (end 138.684 115.2525) (width 0.2) (layer F.Cu) (net 170))
+  (segment (start 138.684 115.2525) (end 139.90498 115.2525) (width 0.2) (layer F.Cu) (net 170))
   (zone (net 2) (net_name GND) (layer F.Cu) (hatch edge 0.508)
     (priority 10)
